Commit message: Update gripper macro

File: urdf/robotiq_3f_gripper.urdf.xacro (robot description, xacro)
@@ -13,4 +13,6 @@
   <link name="world"/>
   <!-- Instantiate the gripper attached to "world" -->
-  <xacro:robotiq_3f_gripper prefix="" parent="world"/>
+  <xacro:robotiq_3f_gripper prefix="" parent="world">
+    <origin xyz="0 0 0" rpy="0 0 0"/>
+  </xacro:robotiq_3f_gripper>
 </robot>

File: urdf/robotiq_3f_gripper_macro.xacro (robot description, xacro)
@@ -11,5 +11,5 @@
       <xacro:robotiq_3f_gripper prefix="gripper_" parent="tool0"/>
   -->
-  <xacro:macro name="robotiq_3f_gripper" params="prefix:='' parent">
+  <xacro:macro name="robotiq_3f_gripper" params="prefix:='' parent *origin">
     <!-- Root frame -->
     <link name="${prefix}robotiq_3f_frame"/>
@@ -17,5 +17,6 @@
       <parent link="${parent}"/>
       <child  link="${prefix}robotiq_3f_frame"/>
-      <origin xyz="0 0 0" rpy="0 0 0"/>
+      <xacro:insert_block name="origin" />
+      <!-- <origin xyz="0 0 0" rpy="0 0 0"/> -->
     </joint>
     <!-- AGS_palm -->
