Commit message: Updated gripper macro

File: urdf/robotiq_3f_gripper_macro.xacro (robot description, xacro)
@@ -39,8 +39,8 @@
       </inertial>
     </link>
-    <joint name="${prefix}robotiq_3f_frame_to_AGS_palm_joint" type="fixed">
-      <parent link="${prefix}robotiq_3f_frame"/>
+    <joint name="${prefix}AGS_wrist_to_AGS_palm_joint" type="fixed">
+      <parent link="${prefix}AGS_wrist"/>
       <child  link="${prefix}AGS_palm"/>
-      <origin xyz="0 0.04127 0" rpy="0 0 0"/>
+      <origin xyz="0 -0.04127 0" rpy="0 1.0432366 3.1415927"/>
     </joint>
     <!-- AGS_finger-base -->
